Commit message: edit URDF robot model

File: Assets/RT605-710-GB/6axis_robot.urdf (robot description, URDF)
Before this commit: robot 6axis_robot, 9 links, 8 joints
Links:
- removed link left_elbow_link
- removed link left_hand_link
- removed link left_shoulder_forward_link
- removed link left_shoulder_link
- removed link left_shoulder_up_link
- removed link left_upper_arm_link
- removed link left_wrist_link
- removed link upper_base_link
- added link arm_link; visual box size=0.1 0.1 0.4
- added link base_link; visual cylinder length=0.15 radius=0.14
- added link elbow_link; visual cylinder length=0.1 radius=0.05
- added link end_link; visual box size=0.03 0.03 0.1
- added link forearm_link; visual box size=0.07 0.07 0.15
- added link hand_link; visual cylinder length=0.05 radius=0.025
- added link shoulder_link; visual box size=0.12 0.12 0.5
- added link upperarm_link; visual box size=0.05 0.05 0.05
- added link upperbase_link; visual cylinder length=0.25 radius=0.1
- added link wrist_link; visual box size=0.05 0.05 0.1
- link torso_link: geometry visual box size=0.05 0.05 0.1
Joints:
- removed joint left_elbow_joint
- removed joint left_hand_joint
- removed joint left_shoulder_forward_joint
- removed joint left_shoulder_joint
- removed joint left_shoulder_up_joint
- removed joint left_upper_arm_joint
- removed joint left_wrist_joint
- added joint arm_joint: type fixed, parent arm_link, child elbow_link, origin xyz=0 0 0.4 rpy=0 0 0
- added joint base_joint: type revolute, parent base_link, child upperbase_link, origin xyz=0 0 0 rpy=0 0 0, axis 0 0 1, limit lower=-2.88 upper=2.88 effort=10 velocity=3
- added joint elbow_joint: type revolute, parent elbow_link, child forearm_link, origin xyz=0 0 0.1 rpy=0 0 0, axis 0 0 1, limit lower=-3.31 upper=3.31 effort=10 velocity=3
- added joint forearm_joint: type revolute, parent forearm_link, child wrist_link, origin xyz=0 0 0.05 rpy=0 0 0, axis 0 1 0, limit lower=-2.01 upper=2.01 effort=10 velocity=3
- added joint hand_joint: type fixed, parent hand_link, child end_link, origin xyz=0 0 0.1 rpy=0 0 0
- added joint shoulder_joint: type fixed, parent shoulder_link, child upperarm_link, origin xyz=0. 0 0.35 rpy=0 -1.57 0
- added joint upperarm_joint: type revolute, parent upperarm_link, child arm_link, origin xyz=0 0 0 rpy=0 0 0, axis 0 1 0, limit lower=-0.96 upper=3.23 effort=10 velocity=3
- added joint upperbase_joint: type fixed, parent upperbase_link, child torso_link, origin xyz=0 0 0.2 rpy=0 0 0
- added joint wrist_joint: type revolute, parent wrist_link, child hand_link, origin xyz=0 0 0.1 rpy=0 0 0, axis 0 0 1, limit lower=-6.28 upper=6.28 effort=10 velocity=3
- joint torso_joint: axis 0 0 1 -> 0 1 0; child torso_link -> shoulder_link; limit lower=-2.88 upper=2.88 effort=10 velocity=3 -> lower=-2.81 upper=1.48 effort=10 velocity=3; origin xyz=0 0 0.05 rpy=0 0 0 -> xyz=0 0 0 rpy=0 0 0; parent upper_base_link -> torso_link
